File: KiCAD/ERK01_PSU_EXT/ERK01_PSU_EXT.kicad_pcb (KiCad board)
At the start: 2 copper layers, 71.1 x 48.3 mm, 6 parts, among them J1 Conn_02x08_Odd_Even, J2 Conn_02x08_Odd_Even, J3 Conn_02x08_Odd_Even, J4 Conn_02x08_Odd_Even, J5 Conn_01x02, J6 Conn_01x03

Commit message: Update: Board Design
Parts:
- added G***: LOGO, myfootprint:Silk_PNPN_Manufactory_600dpi, F.Cu at (182.9, 83.8)
- added J7: Conn_01x03, Connector_JST:JST_XH_B3B-XH-A_1x03_P2.50mm_Vertical, F.Cu at (142.2, 124.5)
- added REF**: MountingHole_3.2mm_M3, MountingHole:MountingHole_3.2mm_M3, F.Cu at (195.6, 124.5)
- added REF**: MountingHole_3.2mm_M3, MountingHole:MountingHole_3.2mm_M3, F.Cu at (129.5, 124.5)
- added REF**: MountingHole_3.2mm_M3, MountingHole:MountingHole_3.2mm_M3, F.Cu at (195.6, 81.3)
- added REF**: MountingHole_3.2mm_M3, MountingHole:MountingHole_3.2mm_M3, F.Cu at (129.5, 81.3)
- J5: value Conn_01x02 -> Conn_02x08_Odd_Even; footprint Connector_JST:JST_XH_B2B-XH-A_1x02_P2.50mm_Vertical -> Connector_IDC:IDC-Header_2x08_P2.54mm_Vertical
- J6: value Conn_01x03 -> Conn_01x02; footprint Connector_JST:JST_XH_B3B-XH-A_1x03_P2.50mm_Vertical -> Connector_JST:JST_XH_B2B-XH-A_1x02_P2.50mm_Vertical
- moved J6 61.4 mm to (137.2, 81.3), turned to 0 degrees
- moved J5 15.5 mm to (195.6, 111.8), turned to 180 degrees
Connections:
- J5 pad 1: /+5V -> /-12V
- J5 pad 2: GND -> /-12V
- J6 pad 1: /+12V -> /+5V
Routing:
- net GND: track 116.9 -> 160.2 mm, vias 0 -> 4
- net /+5V: track 62.0 -> 88.5 mm
- net /+12V: track 63.1 -> 86.4 mm, vias 0 -> 2
- net /-12V: track 61.0 -> 77.4 mm
- net /Gate: track 48.3 -> 63.5 mm
- net /CV: track 48.3 -> 63.5 mm
