File: KiCAD/ERK01_PSU_EXT_Ver.1.1/ERK01_PSU_EXT.sch (KiCad schematic (older format))
At the start: 23 parts, among them J1 Conn_02x08_Odd_Even, J2 Conn_02x08_Odd_Even, J3 Conn_02x08_Odd_Even, J4 Conn_02x08_Odd_Even, J5 Conn_02x08_Odd_Even, J6 +5V, J7 +-12V

Commit message: Gerber
Parts:
- removed J? (x2): +5V, Connector_JST:JST_XH_B2B-XH-A_1x02_P2.50mm_Vertical, symbol Connector_Generic:Conn_01x02
- removed J? (x2): +-12V, Connector_JST:JST_XH_B3B-XH-A_1x03_P2.50mm_Vertical, symbol Connector_Generic:Conn_01x03
- added H1, H2, H3, H4: MountingHole, MountingHole:MountingHole_3.2mm_M3, symbol Mechanical:MountingHole
- D1, D2, D3: renamed from D?; footprint (none) -> LED_THT:LED_D3.0mm
- R1, R2, R3: renamed from R?; footprint (none) -> Resistor_THT:R_Axial_DIN0207_L6.3mm_D2.5mm_P7.62mm_Horizontal
- gave numbers to parts that had none: 6
- renumbered J7 to J13, J6 to J8
Connections:
- net +12V: now also D2.2 (A); no longer R2.2
- net +5V: now also D1.2 (A); no longer R1.2
- net -12V: now also D3.2 (A); no longer R3.2
- net GND: now also R1.1, R2.1, R3.1; no longer D1.1 (K), D2.1 (K), D3.1 (K)
- new net: D1.1 (K), R1.2
- new net: D2.1 (K), R2.2
- new net: D3.1 (K), R3.2
Other:
- moved on the sheet: D1, D2, D3, R1, R2, R3

Commit message: Bug fixed
Connections:
- net -12V: now also D3.1 (K); no longer D3.2 (A)
- net at R3.2: now also D3.2 (A); no longer D3.1 (K)
Other:
- moved on the sheet: D3
Changed lines of the file:
@@
 F 3 "~" H 5300 4650 50  0001 C CNN
 	1    5300 4650
-	-1   0    0    1
+	1    0    0    -1
 $EndComp
 Text Label 4950 3950 0    50   ~ 0
